File: power-supply/kicad/psu.sch (KiCad schematic (older format))
At the start: 25 parts

Commit message: Current Sources
Parts:
- added D?: LED, symbol Device:LED_ALT
- added Q?: NPN, symbol Device:Q_NPN_BCE
- added R: R_POT, symbol Device:R_POT
- added R1: R1, symbol Device:R
- added R?: R2, symbol Device:R
- added U?: LM317, Package_TO_SOT_THT:TO-220-3_Vertical, symbol Regulator_Linear:LM317_TO-220
- added U?: Load, symbol load:Load
Connections:
- net labels added: I_limit
- wire segments 65 -> 89
Other:
- note added: "1.25\n= ---\n R"
- note added: "Current Limiter"
- note added: "I"
- note added: "LED Current Source"
- note added: "limit"
Changed lines of the file:
@@
 	0    -1   -1   0
 $EndComp
-Text GLabel 1250 2650 0    50   Input ~ 0
+Text GLabel 1200 2650 0    50   Input ~ 0
 Vin
+$Comp
+L Regulator_Linear:LM317_TO-220 U?
+U 1 1 6592B61E
+P 3650 2850
+F 0 "U?" H 3650 3092 50  0001 C CNN
+F 1 "LM317" H 3650 3001 50  0000 C CNN
+F 2 "Package_TO_SOT_THT:TO-220-3_Vertical" H 3650 3100 50  0001 C CIN
+F 3 "http://www.ti.com/lit/ds/symlink/lm317.pdf" H 3650 2850 50  0001 C CNN
+	1    3650 2850
+	1    0    0    -1
+$EndComp
+Wire Wire Line
+	3200 2850 3350 2850
+Text GLabel 3200 2850 0    50   Input ~ 0
+Vin
+$Comp
+L Device:R_POT R
+U 1 1 6592D3CC
+P 4250 2850
+F 0 "R" V 4135 2850 50  0000 C CNN
+F 1 "R_POT" V 4135 2850 50  0001 C CNN
+F 2 "" H 4250 2850 50  0001 C CNN
+F 3 "~" H 4250 2850 50  0001 C CNN
+	1    4250 2850
+	0    -1   -1   0
+$EndComp
+Text GLabel 4650 2850 2    50   Output ~ 0
+I_limit
+Wire Wire Line
+	4650 2850 4500 2850
+Wire Wire Line
+	3950 2850 4000 2850
+Wire Wire Line
+	4000 2850 4000 2650
+Wire Wire Line
+	4000 2650 4250 2650
+Wire Wire Line
+	4250 2650 4250 2700
+Connection ~ 4000 2850
+Wire Wire Line
+	4000 2850 4100 2850
+Wire Wire Line
+	3650 3150 3650 3200
+Wire Wire Line
+	3650 3200 4500 3200
+Wire Wire Line
+	4500 3200 4500 2850
+Connection ~ 4500 2850
+Wire Wire Line
+	4500 2850 4400 2850
+Text Notes 4650 3100 0    79   ~ 0
+I
+Text Notes 4700 3150 0    39   ~ 0
+limit
+Text Notes 4850 3150 0    39   ~ 0
+   1.25\n= ---\n     R
+Text Notes 3800 3550 0    39   ~ 0
+Current Limiter
+$Comp
+L Device:R R1
+U 1 1 6593C804
+P 1650 5200
+F 0 "R1" H 1720 5246 50  0001 L CNN
+F 1 "R1" H 1720 5200 50  0000 L CNN
+F 2 "" V 1580 5200 50  0001 C CNN
+F 3 "~" H 1650 5200 50  0001 C CNN
+	1    1650 5200
+	1    0    0    -1
+$EndComp
+Wire Wire Line
+	1400 4600 1650 4600
+Wire Wire Line
+	1650 4600 1650 5050
+$Comp
+L power:GND #PWR?
+U 1 1 6593C80C
+P 1650 6150
+F 0 "#PWR?" H 1650 5900 50  0001 C CNN
+F 1 "GND" H 1655 5977 50  0000 C CNN
+F 2 "" H 1650 6150 50  0001 C CNN
+F 3 "" H 1650 6150 50  0001 C CNN
+	1    1650 6150
+	1    0    0    -1
+$EndComp
+Wire Wire Line
+	1650 6000 1650 6100
+Wire Wire Line
+	1650 5350 1650 5550
+$Comp
+L Device:LED_ALT D?
+U 1 1 6593C814
+P 1650 5850
+F 0 "D?" V 1689 5732 50  0001 R CNN
+F 1 "LED" V 1643 5732 50  0000 R CNN
+F 2 "" H 1650 5850 50  0001 C CNN
+F 3 "~" H 1650 5850 50  0001 C CNN
+	1    1650 5850
+	0    -1   -1   0
+$EndComp
+Text GLabel 1400 4600 0    50   Input ~ 0
+Vin
+$Comp
+L load:Load U?
+U 1 1 6593E468
+P 3150 4350
+F 0 "U?" H 3328 3846 50  0001 L CNN
+F 1 "Load" H 3000 3800 50  0000 L CNN
+F 2 "" H 3150 4350 50  0001 C CNN
+F 3 "" H 3150 4350 50  0001 C CNN
+	1    3150 4350
+	1    0    0    -1
+$EndComp
+$Comp
+L Device:Q_NPN_BCE Q?
+U 1 1 6593F45A
+P 2400 5550
+F 0 "Q?" H 2591 5596 50  0000 L CNN
+F 1 "NPN" H 2591 5505 50  0000 L CNN
+F 2 "" H 2600 5650 50  0001 C CNN
+F 3 "~" H 2400 5550 50  0001 C CNN
+	1    2400 5550
+	1    0    0    -1
+$EndComp
+$Comp
+L Device:R R?
+U 1 1 65940643
+P 2500 5900
+F 0 "R?" H 2570 5946 50  0001 L CNN
+F 1 "R2" H 2570 5900 50  0000 L CNN
+F 2 "" V 2430 5900 50  0001 C CNN
+F 3 "~" H 2500 5900 50  0001 C CNN
+	1    2500 5900
+	1    0    0    -1
+$EndComp
+Wire Wire Line
+	2500 5350 2500 5250
+Wire Wire Line
+	1650 4600 3100 4600
+Connection ~ 1650 4600
+Wire Wire Line
+	2500 6050 2500 6100
+Wire Wire Line
+	2500 6100 1650 6100
+Connection ~ 1650 6100
+Wire Wire Line
+	1650 6100 1650 6150
+Connection ~ 1650 5550
+Wire Wire Line
+	1650 5550 1650 5700
+Wire Wire Line
+	1650 5550 2200 5550
+Wire Wire Line
+	2500 5250 3100 5250
+Wire Wire Line
+	3100 5250 3100 5200
+Text Notes 2150 6650 0    39   ~ 0
+LED Current Source
 $EndSCHEMATC

Commit message: decoupling capacitor
Parts:
- added C5: 100 nF, Capacitor_SMD:C_0805_2012Metric, symbol Device:C_Small
- added J1: Conn_01x02_Male, Connector_PinSocket_2.54mm:PinSocket_1x02_P2.54mm_Vertical, symbol Connector:Conn_01x02_Male
- added U7: ATtiny1614-SS, Package_SO:SOIC-14_3.9x8.7mm_P1.27mm, symbol MCU_Microchip_ATtiny:ATtiny1614-SS
- gave numbers to parts that had none: 30
- renumbered R to R4
Connections:
- net GND: now also C5.1, J1.2 (Pin_2), U7.14 (GND)
- new net VCC: C5.2, J1.1 (Pin_1), U7.1 (VCC)
